Commit message: trochę inwencji twórczej

File: urdf_steer/urdf/robot.urdf (robot description, URDF)
Before this commit: robot firstRobot, 5 links, 4 joints
Links:
- link link_1: geometry visual box size=${l_width} ${l_width} ${params['i1']['l_len']}
- link link_2: geometry visual box size=${l_width} ${l_width} ${params['i2']['l_len']}
- link link_3: geometry visual box size=${l_width} ${l_width} ${params['i3']['l_len']}
Joints:
- joint base_to_link1: axis 0 0 1 -> (none); limit lower=-1 upper=0 effort=1000.0 velocity=1 -> (none); origin xyz=${props['i1']['j_xyz']} rpy=${props['i1']['j_rpy']} -> xyz=${params['i1']['j_xyz']} rpy=${params['i1']['j_rpy']}
- joint link1_to_link2: axis 0 0 1 -> (none); limit lower=-1 upper=0 effort=1000.0 velocity=1 -> (none); origin xyz=${props['i2']['j_xyz']} rpy=${props['i2']['j_rpy']} -> xyz=${params['i2']['j_xyz']} rpy=${params['i2']['j_rpy']}
- joint link2_to_link3: axis 0 0 1 -> (none); limit lower=-1 upper=0 effort=1000.0 velocity=1 -> (none); origin xyz=${props['i3']['j_xyz']} rpy=${props['i3']['j_rpy']} -> xyz=${params['i3']['j_xyz']} rpy=${params['i3']['j_rpy']}

Commit message: Przynajmniej działa

File: urdf_steer/urdf/robot.urdf (robot description, URDF)
Before this commit: robot firstRobot, 5 links, 4 joints
Links:
- link hand: geometry visual box size=${l_width} ${l_width} ${l_width}
- link link_1: geometry visual box size=${l_width} ${l_width} ${params['i2']['l_len']}
- link link_2: geometry visual box size=${l_width} ${l_width} ${params['i3']['l_len']}
- link link_3: geometry visual box size=${l_width} ${l_width} 1

File: urdf_steer/urdf/robot_movable.urdf (robot description, URDF)
Before this commit: robot forstRobot, 5 links, 4 joints
Links:
- link link_1: geometry visual box size=${l_width} ${l_width} ${params['i2']['l_len']}
- link link_2: geometry visual box size=${l_width} ${l_width} ${params['i3']['l_len']}
- link link_3: geometry visual box size=${l_width} ${l_width} 1
Joints:
- joint link2_to_link3: type prismatic -> continuous

Commit message: Lekka zmiana

File: urdf_steer/urdf/robot.urdf (robot description, URDF)
Before this commit: robot firstRobot, 5 links, 4 joints
Links:
- link link_3: geometry visual box size=${l_width} ${l_width} ${params['hand']['l_len']}
Joints:
- joint link3_to_hand: origin xyz=0 0 0 rpy=0 0 0 -> xyz=${params['hand']['j_xyz']} rpy=${params['hand']['j_rpy']}

File: urdf_steer/urdf/robot_movable.urdf (robot description, URDF)
Before this commit: robot forstRobot, 5 links, 4 joints
Links:
- link link_3: geometry visual box size=${l_width} ${l_width} ${params['hand']['l_len']}
Joints:
- joint link3_to_hand: origin xyz=0 0 0 rpy=0 0 0 -> xyz=${params['hand']['j_xyz']} rpy=${params['hand']['j_rpy']}
