Commit message: Dodano restrykcje

File: lab3/urdf/robot_movable.urdf (robot description, URDF)
Before this commit: robot forstRobot, 5 links, 4 joints
Joints:
- joint base_to_link1: limit lower=-1 upper=0 effort=1000.0 velocity=1 -> lower=-1.57079632679 upper=1.57079632679 effort=1000.0 velocity=1; type continuous -> revolute
- joint link1_to_link2: limit lower=-1 upper=0 effort=1000.0 velocity=1 -> lower=-1.57079632679 upper=1.57079632679 effort=1000.0 velocity=1; type continuous -> revolute
- joint link2_to_link3: limit lower=-1 upper=0 effort=1000.0 velocity=1 -> lower=-1.57079632679 upper=0 effort=1000.0 velocity=1; type continuous -> revolute

Commit message: Zwiększono zakres ruchu robota

File: lab3/urdf/robot_movable.urdf (robot description, URDF)
Before this commit: robot forstRobot, 5 links, 4 joints
Joints:
- joint base_to_link1: limit lower=-1.57079632679 upper=1.57079632679 effort=1000.0 velocity=1 -> lower=-2 upper=2 effort=1000.0 velocity=1
- joint link1_to_link2: limit lower=-1.57079632679 upper=1.57079632679 effort=1000.0 velocity=1 -> lower=-2 upper=2 effort=1000.0 velocity=1
- joint link2_to_link3: limit lower=-1.57079632679 upper=0 effort=1000.0 velocity=1 -> lower=-2 upper=1 effort=1000.0 velocity=1
