Commit message: popraweczki, ale chyba już wszystko gitesik

File: lab5/urdf/robot_movable.urdf (robot description, URDF)
Before this commit: robot forstRobot, 5 links, 4 joints
Joints:
- joint base_to_link1: type continuous -> revolute
- joint link1_to_link2: type continuous -> revolute
- joint link2_to_link3: type continuous -> revolute
